File: IMU_BB_Rev2/IMU_BB_Rev2.kicad_pcb (KiCad board)
At the start: 2 copper layers, 12.7 x 12.7 mm, 10 parts, among them J1 Conn_01x04, U1 BMI270

Commit message: Update IMU_BB_Rev2.kicad_pcb
Other:
- board text added: "TP SCL"
Changed lines of the file:
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@@
   )
   (gr_rect (start 68.235 52.74) (end 80.945 65.45) (layer "Edge.Cuts") (width 0.1) (fill none))
+  (gr_text "TP SCL" (at 68.98 57.05 90) (layer "F.SilkS")
+    (effects (font (size 0.2 0.2) (thickness 0.05)))
+  )
   (gr_text "TP 3.3V" (at 76.54 65.14) (layer "F.SilkS")
     (effects (font (size 0.2 0.2) (thickness 0.05)))
@@
   )
   (gr_text "Test Board\n-Kylie Angel" (at 78.06 57.07) (layer "F.SilkS")
-    (effects (font (size 0.3 0.3) (thickness 0.06)))
+    (effects (font (size 0.25 0.25) (thickness 0.05)))
   )
   (gr_text "+3.3V" (at 76.05 52.96) (layer "F.SilkS")

Commit message: redid PCB
Parts:
- moved TP2 9.61 mm to (69.8, 64.2), turned to -90 degrees
- moved TP4 7.27 mm to (69.8, 58.0), turned to -90 degrees
- moved TP1 7.07 mm to (69.8, 62.0), turned to -90 degrees
- moved R1 5.35 mm to (75.7, 58.5), turned to 0 degrees
- moved R2 3.03 mm to (72.3, 58.5)
- moved TP3 3.00 mm to (69.8, 60.0), turned to -90 degrees
- moved U1 1.89 mm to (74.2, 61.8)
- moved C1 1.70 mm to (79.9, 61.7)
- moved C2 1.63 mm to (77.8, 61.7)
- moved J1 0.59 mm to (78.4, 55.0)
Routing:
- net /IMU_A_SDA: track 26.4 -> 11.0 mm
- net +3V3: track 31.5 -> 25.2 mm
- net GND: track 13.4 -> 7.54 mm, vias 4 -> 3
- net /IMU_A_SCL: track 13.0 -> 17.8 mm
- added copper zone on F.Cu, net +3V3
Other:
- board text added: "Test Soldering Board UtProsat Space@VT Kylie Angel"
- board text removed: "Test Board -Kylie Angel"
