File: IMU_BB_Rev2/IMU_BB_Rev2.kicad_sch (KiCad schematic)
At the start: 10 parts, among them J1 Conn_01x04, U1 BMI270

Commit message: redid PCB
Changed lines of the file:
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@@
+    (stroke (width 0) (type default) (color 0 0 0 0))
+  )
+  (wire (pts (xy 36.83 97.79) (xy 45.72 97.79))
     (stroke (width 0) (type default) (color 0 0 0 0))
   )
@@
     (stroke (width 0) (type default) (color 0 0 0 0))
   )
-  (wire (pts (xy 38.1 97.79) (xy 45.72 97.79))
-    (stroke (width 0) (type default) (color 0 0 0 0))
-  )
   (wire (pts (xy 111.633 36.068) (xy 111.633 37.211))
     (stroke (width 0) (type default) (color 0 0 0 0))
@@
     (stroke (width 0) (type default) (color 0 0 0 0))
   )
-  (wire (pts (xy 38.1 95.25) (xy 45.72 95.25))
-    (stroke (width 0) (type default) (color 0 0 0 0))
-  )
   (polyline (pts (xy 129.667 21.59) (xy 20.32 21.59))
     (stroke (width 0) (type default) (color 0 0 0 0))
@@
     (stroke (width 0) (type default) (color 0 0 0 0))
   )
+  (wire (pts (xy 36.83 95.25) (xy 45.72 95.25))
+    (stroke (width 0) (type default) (color 0 0 0 0))
+  )
   (wire (pts (xy 41.91 49.911) (xy 62.738 49.911))
     (stroke (width 0) (type default) (color 0 0 0 0))
@@
     (effects (font (size 1.27 1.27)) (justify right))
   )
-  (hierarchical_label "IMU_A_SCL" (shape input) (at 38.1 95.25 180)
+  (hierarchical_label "IMU_A_SCL" (shape input) (at 36.83 95.25 180)
     (effects (font (size 1.27 1.27)) (justify right))
   )
@@
     (effects (font (size 1.27 1.27)) (justify left))
   )
-  (hierarchical_label "IMU_A_SDA" (shape input) (at 38.1 97.79 180)
+  (hierarchical_label "IMU_A_SDA" (shape input) (at 36.83 97.79 180)
     (effects (font (size 1.27 1.27)) (justify right))
   )
